File: kicad/bmw-e36-abs-adapter.kicad_sch (KiCad schematic)
At the start: 41 parts, among them J1 TE_9-6437287-8, J2 SWD, U1 TPSM33610S5, U2 TLE42744DV33ATMA1, U3 STM32F042K6Ux, Y1 ECS-160-10-36Q-AES-TR

Commit message: PCB Design WIP
Parts:
- renumbered TP2 to TP1, TP3 to TP2, TP1 to TP3
